Commit message: Add detailed KIWI camera catalog and simulation parameter manifests

File: models/x5/urdf/insta360_x5.urdf (robot description, URDF)
Before this commit: robot insta360_x5, 4 links, 3 joints
Joints:
- joint x5_front_lens_surface_fixed: origin xyz=0.0191 0 0.10400000000000001 rpy=0 0 0 -> xyz=0.0191 0 0.10400000000000001 rpy=-1.57079632679 0 -1.57079632679
- joint x5_rear_lens_surface_fixed: origin xyz=-0.0191 0 0.10400000000000001 rpy=0 0 0 -> xyz=-0.0191 0 0.10400000000000001 rpy=-1.57079632679 0 1.57079632679
